Commit message: Update file permissions and enhance .gitignore
- Changed file permissions for multiple files to make them executable.
- Updated .gitignore to include additional build outputs and Python-related files.
- Added new README content for URDF and Robot State Publisher usage.
- Added images and updated links in various directories.
- Ensured consistency in naming conventions within URDF files.

File: URDF/mybot.urdf (robot description, URDF)
Before this commit: robot my_custom_bot, 6 links, 5 joints
Links:
- removed link base-footprint
- removed link front-caster-wheel
- removed link rear-left-wheel-link
- removed link rear-right-wheel-link
- added link base_footprint
- added link front_caster_wheel; visual sphere radius=0.05
- added link rear_left_wheel_link; visual cylinder length=0.05 radius=0.1
- added link rear_right_wheel_link; visual cylinder length=0.05 radius=0.1
Joints:
- removed joint base-footprint-joint
- removed joint base-front-caster-wheel-joint
- removed joint base-lidar-joint
- removed joint base-rear-left-wheel-joint
- removed joint base-rear-right-wheel-joint
- added joint base_front_caster_wheel_joint: type continuous, parent base_link, child front_caster_wheel, origin xyz=-0.15 0 -0.05 rpy=0 0 0, axis 0 0 1
- added joint base_joint: type fixed, parent base_footprint, child base_link, origin xyz=0 0 0 rpy=0 0 0
- added joint base_lidar_joint: type fixed, parent base_link, child lidar_link, origin xyz=0 0 0.225 rpy=0 0 0
- added joint base_rear_left_wheel_joint: type continuous, parent base_link, child rear_left_wheel_link, origin xyz=0.15 0.2 0 rpy=0 0 0, axis 0 1 0
- added joint base_rear_right_wheel_joint: type continuous, parent base_link, child rear_right_wheel_link, origin xyz=0.15 -0.2 0 rpy=0 0 0, axis 0 1 0
